File: karifa.kicad_pcb (KiCad board)
At the start: 2 copper layers, 27 parts, among them J1 Conn_01x04, SW1 SW_DPST_x2, U1 STC8G1K08-SOP16

Commit message: proto nyak
Parts:
- BT1: moved to B.Cu
- moved D11 67.7 mm to (227.1, 25.5), turned to 180 degrees
- moved D10 65.5 mm to (223.3, 25.5)
- moved D9 64.6 mm to (227.1, 30.6), turned to 180 degrees
- moved D5 62.9 mm to (227.1, 40.7), turned to 180 degrees
- moved D3 56.3 mm to (227.3, 45.7), turned to 180 degrees
- moved R1 49.9 mm to (196.2, 43.8), turned to 180 degrees
- moved R2 45.7 mm to (196.2, 46.4), turned to 180 degrees
- moved BT1 45.5 mm to (227.3, 52.1), turned to 180 degrees
- moved R3 45.1 mm to (196.2, 48.9), turned to 180 degrees
- moved R9 44.3 mm to (207.6, 41.3), turned to -90 degrees
- moved C1 43.8 mm to (208.9, 47.6), turned to 90 degrees
- moved D2 42.0 mm to (223.5, 45.7)
- moved R8 41.7 mm to (222.1, 28.0), turned to 180 degrees
- moved D13 40.8 mm to (205.1, 38.1)
- moved D1 40.8 mm to (202.6, 45.7)
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Connections:
- J1 pad 3: unconnected-(J1-Pad3) -> /P3.1
- U1 pad 6: unconnected-(U1-Pad6) -> VCC
- U1 pad 8: unconnected-(U1-Pad8) -> GND
Routing:
- net /MPX1: track 0.00 -> 64.5 mm
- net /MPX2: track 0.00 -> 51.0 mm
- net GND: track 0.00 -> 33.3 mm
- net Net-(SW1-Pad1): track 0.00 -> 22.7 mm
- net VCC: track 0.00 -> 19.3 mm
- net /P3.7: track 0.00 -> 13.6 mm
- net /P3.6: track 0.00 -> 10.5 mm
- net Net-(D1-Pad5): track 0.00 -> 7.28 mm
- net Net-(D1-Pad6): track 0.00 -> 7.10 mm
- net Net-(D1-Pad4): track 0.00 -> 7.10 mm
- net /P3.5: track 0.00 -> 7.02 mm
- net /P3.1: track 0.00 -> 6.35 mm
- net /P3.3: track 0.00 -> 5.81 mm
- net Net-(D2-Pad2): track 0.00 -> 5.15 mm
- net Net-(D4-Pad2): track 0.00 -> 5.07 mm
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
Commit message: karifa outline
Parts:
- BT1: moved to F.Cu
- moved D11 68.7 mm to (206.1, 90.8), turned to 0 degrees
- moved D10 66.6 mm to (210.5, 90.8)
- moved D9 65.4 mm to (201.6, 90.8), turned to 0 degrees
- moved D5 63.4 mm to (188.2, 90.8), turned to 0 degrees
- moved D3 56.8 mm to (192.7, 90.8), turned to 0 degrees
- moved R1 51.3 mm to (214.9, 91.6), turned to 0 degrees
- moved R2 47.1 mm to (232.3, 76.6), turned to 0 degrees
- moved R3 46.2 mm to (239.5, 65.2), turned to 0 degrees
- moved R9 45.7 mm to (227.1, 82.7), turned to 0 degrees
- moved BT1 45.5 mm to (188.0, 75.0), turned to 0 degrees
- moved C1 44.7 mm to (197.1, 90.8), turned to 0 degrees
- moved D2 43.2 mm to (218.8, 88.6)
- moved R8 43.1 mm to (243.9, 65.2), turned to 0 degrees
- moved D13 42.3 mm to (227.9, 73.7)
- moved D1 42.2 mm to (220.7, 83.8)
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Routing:
- net /MPX1: track 64.5 -> 0.00 mm
- net /MPX2: track 51.0 -> 0.00 mm
- net GND: track 33.3 -> 0.00 mm
- net Net-(SW1-Pad1): track 22.7 -> 0.00 mm
- net VCC: track 19.3 -> 0.00 mm
- net /P3.7: track 13.6 -> 0.00 mm
- net /P3.6: track 10.5 -> 0.00 mm
- net Net-(D1-Pad5): track 7.28 -> 0.00 mm
- net Net-(D1-Pad6): track 7.10 -> 0.00 mm
- net Net-(D1-Pad4): track 7.10 -> 0.00 mm
- net /P3.5: track 7.02 -> 0.00 mm
- net /P3.1: track 6.35 -> 0.00 mm
- net /P3.3: track 5.81 -> 0.00 mm
- net Net-(D2-Pad2): track 5.15 -> 0.00 mm
- net Net-(D4-Pad2): track 5.07 -> 0.00 mm
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Other:
- board outline added: 38.2 x 54.8 mm

Commit message: nyakterv majdnem kesz
Parts:
- added L1: L, Inductor_SMD:L_1008_2520Metric, F.Cu at (128.5, 58.9)
- added L2: L, Inductor_SMD:L_1008_2520Metric, F.Cu at (130.2, 55.2)
- added L3: L, Inductor_SMD:L_1008_2520Metric, F.Cu at (131.8, 58.9)
- added Q1: AO3401A, Package_TO_SOT_SMD:SOT-23, F.Cu at (128.0, 64.3)
- added Q2: AO3401A, Package_TO_SOT_SMD:SOT-23, F.Cu at (123.2, 75.2)
- added Q3: AO3401A, Package_TO_SOT_SMD:SOT-23, F.Cu at (132.2, 64.3)
- BT1: footprint Battery:BatteryHolder_ComfortableElectronic_CH273-2450_1x2450 -> karifa:CR2032_Holder; moved to B.Cu
- D1: value LED_RGB -> LED_ARGB; footprint LED_SMD:LED_RGB_5050-6 -> LED_SMD:LED_RGB_Wuerth-PLCC4_3.2x2.8mm_150141M173100
- J1: footprint Connector_PinHeader_2.54mm:PinHeader_1x04_P2.54mm_Vertical -> Connector_PinHeader_1.27mm:PinHeader_1x04_P1.27mm_Vertical
- R1, R2, R3, R4, R5, R6, R7, R8, R9: footprint Resistor_SMD:R_0805_2012Metric -> Resistor_SMD:R_0603_1608Metric
- moved D12 117.6 mm to (125.7, 91.6)
- moved R3 116.6 mm to (124.2, 83.2)
- moved D6 111.5 mm to (116.5, 81.2)
- moved R6 109.2 mm to (136.1, 79.2), turned to 180 degrees
- moved D4 109.1 mm to (115.2, 90.0)
- moved R8 108.3 mm to (136.1, 75.8), turned to 180 degrees
- moved R2 108.1 mm to (124.2, 78.9), turned to -90 degrees
- moved U1 104.0 mm to (130.2, 82.0)
- moved R7 103.8 mm to (136.1, 77.5), turned to 180 degrees
- moved R9 103.0 mm to (124.2, 81.5)
- moved D8 100.6 mm to (123.1, 64.0)
- moved D2 99.0 mm to (125.8, 55.0)
- moved R4 96.7 mm to (136.1, 82.8), turned to 180 degrees
- moved D1 96.2 mm to (130.0, 51.8), turned to 180 degrees
- moved D13 95.3 mm to (134.3, 91.6), turned to 180 degrees
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Connections:
- D1 pad 1: Net-(D1-Pad1) -> GND
- D1 pad 2: Net-(D1-Pad2) -> Net-(L2-Pad1)
- D1 pad 3: Net-(D1-Pad3) -> Net-(L3-Pad1)
- R1 pad 1: Net-(D1-Pad1) -> VCC
- R1 pad 2: GND -> /P5.5
- R2 pad 1: Net-(D1-Pad2) -> VCC
- R2 pad 2: GND -> /P1.6
- R3 pad 1: Net-(D1-Pad3) -> VCC
- R3 pad 2: GND -> /P5.4
- R9 pad 2: /P1.6 -> /P1.7
- U1 pad 4: Net-(D1-Pad6) -> /P1.7
- U1 pad 5: Net-(D1-Pad5) -> /P5.4
- U1 pad 7: Net-(D1-Pad4) -> /P5.5
Routing:
- net /MPX2: track 0.00 -> 78.5 mm, vias 0 -> 2
- net /MPX1: track 0.00 -> 76.3 mm, vias 0 -> 2
- net VCC: track 0.00 -> 56.3 mm, vias 0 -> 5
- net Net-(D2-Pad2): track 0.00 -> 55.4 mm, vias 0 -> 2
- net Net-(D10-Pad2): track 0.00 -> 43.1 mm, vias 0 -> 2
- net Net-(D4-Pad2): track 0.00 -> 41.0 mm, vias 0 -> 2
- net Net-(D6-Pad2): track 0.00 -> 36.2 mm, vias 0 -> 2
- net Net-(L2-Pad1): track 0.00 -> 28.2 mm, vias 0 -> 2
- net Net-(D8-Pad2): track 0.00 -> 28.0 mm, vias 0 -> 2
- net /P5.5: track 0.00 -> 24.5 mm, vias 0 -> 2
- net /P5.4: track 0.00 -> 22.7 mm, vias 0 -> 2
- net Net-(D12-Pad2): track 0.00 -> 19.5 mm, vias 0 -> 2
- net Net-(D1-Pad4): track 0.00 -> 19.1 mm
- net Net-(L3-Pad1): track 0.00 -> 13.6 mm
- net Net-(SW1-Pad1): track 0.00 -> 12.8 mm, vias 0 -> 2
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- added copper zone on F.Cu, net GND

Commit message: nyakterv haladas
Parts:
- added C2: 10uF, Capacitor_SMD:C_0805_2012Metric, F.Cu at (133.3, 96.3)
- added C3: 10uF, Capacitor_SMD:C_0805_2012Metric, F.Cu at (127.0, 96.3)
- C1: value C -> 100nF
- R1, R2, R3: value R -> 100k
- R4, R5, R6, R7, R8, R9: value R -> 1k
- moved L2 0.26 mm to (130.2, 55.0)
Routing:
- net GND: track 1.89 -> 119.0 mm, vias 0 -> 12
- net Net-(SW1-Pad1): track 12.8 -> 30.6 mm
- net VCC: track 56.3 -> 69.6 mm, vias 5 -> 4
- net Net-(D8-Pad2): track 28.0 -> 34.1 mm
- net Net-(D12-Pad2): track 19.5 -> 25.3 mm
- net Net-(D2-Pad2): track 55.4 -> 49.6 mm
- net /MPX1: track 76.3 -> 81.9 mm
- net /P5.4: track 22.7 -> 28.0 mm
- net Net-(D6-Pad2): track 36.2 -> 40.3 mm
- net /MPX2: track 78.5 -> 81.5 mm
- net /P5.5: track 24.5 -> 27.0 mm
- net Net-(D1-Pad2): track 28.2 -> 30.3 mm
- net Net-(D4-Pad2): track 41.0 -> 41.7 mm
- added copper zone on B.Cu, net GND
