File: karifa.kicad_pcb (KiCad board)
At the start: 2 copper layers, 38.2 x 54.8 mm, 45 parts, among them J1 Conn_01x04, Q1 AO3401A, Q2 AO3401A, Q3 AO3401A, SW1 SW_DPST_x2, T1 Tab, U1 STC8G1K08-SOP16

Commit message: Fixed some stuff in repo + additional tab so that the guys at JLCPCB will be happy.
Parts:
- added T1: Tab, kikit:Tab, F.Cu at (147.3, 71.6)
- added T1: Tab, kikit:Tab, F.Cu at (111.8, 71.6)
Changed lines of the file:
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@@
     )
+  )
+  (footprint "kikit:Tab" (layer "F.Cu")
+    (at 147.32 71.58 180)
+    (descr "A symbol representing annotation for tab placement")
+    (property "Sheetfile" "karifa.kicad_sch")
+    (property "Sheetname" "")
+    (property "exclude_from_bom" "")
+    (attr exclude_from_pos_files exclude_from_bom)
+    (fp_text reference "T1" (at 0 -2) (layer "F.SilkS") hide
+      (effects (font (size 1 1) (thickness 0.15)))
+    )
+    (fp_text value "Tab" (at -2.75 -1) (layer "Dwgs.User")
+      (effects (font (size 1.2 1.2) (thickness 0.2)))
+    )
+    (fp_text user "KIKIT: width: 1.9mm" (at -5.5 0 90) (layer "Dwgs.User")
+      (effects (font (size 1 1) (thickness 0.15)))
+    )
+    (fp_line (start 0.25 0) (end -0.75 -1) (layer "Dwgs.User") (width 0.3))
+    (fp_line (start 0.25 1) (end 0.25 -1) (layer "Dwgs.User") (width 0.3))
+    (fp_line (start 0.25 0) (end -2.75 0) (layer "Dwgs.User") (width 0.3))
+    (fp_line (start 0.25 0) (end -0.75 1) (layer "Dwgs.User") (width 0.3))
   )
   (footprint "LED_SMD:LED_0805_2012Metric" (layer "F.Cu")
@@
     )
   )
+  (footprint "kikit:Tab" (layer "F.Cu")
+    (at 111.76 71.58)
+    (descr "A symbol representing annotation for tab placement")
+    (property "Sheetfile" "karifa.kicad_sch")
+    (property "Sheetname" "")
+    (property "exclude_from_bom" "")
+    (attr exclude_from_pos_files exclude_from_bom)
+    (fp_text reference "T1" (at 0 -2) (layer "F.SilkS") hide
+      (effects (font (size 1 1) (thickness 0.15)))
+    )
+    (fp_text value "Tab" (at -2.75 -1) (layer "Dwgs.User")
+      (effects (font (size 1.2 1.2) (thickness 0.2)))
+    )
+    (fp_text user "KIKIT: width: 1.9mm" (at -5.5 0 90) (layer "Dwgs.User")
+      (effects (font (size 1 1) (thickness 0.15)))
+    )
+    (fp_line (start 0.25 1) (end 0.25 -1) (layer "Dwgs.User") (width 0.3))
+    (fp_line (start 0.25 0) (end -0.75 -1) (layer "Dwgs.User") (width 0.3))
+    (fp_line (start 0.25 0) (end -2.75 0) (layer "Dwgs.User") (width 0.3))
+    (fp_line (start 0.25 0) (end -0.75 1) (layer "Dwgs.User") (width 0.3))
+  )
   (footprint "LED_SMD:LED_0805_2012Metric" (layer "F.Cu")
     (at 125.75 55)
@@
     )
     (fp_line (start 0.25 0) (end -0.75 -1) (layer "Dwgs.User") (width 0.3))
+    (fp_line (start 0.25 0) (end -2.75 0) (layer "Dwgs.User") (width 0.3))
     (fp_line (start 0.25 1) (end 0.25 -1) (layer "Dwgs.User") (width 0.3))
-    (fp_line (start 0.25 0) (end -2.75 0) (layer "Dwgs.User") (width 0.3))
     (fp_line (start 0.25 0) (end -0.75 1) (layer "Dwgs.User") (width 0.3))
   )

Commit message: Sent to fab.
Other:
- board text added: "PCB by Dávid Warranty void if you can read this. Vesztettem"
- board text added: "Rev.A"
Changed lines of the file:
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@@
     (property "Sheetname" "")
     (attr smd)
-    (fp_text reference "D9" (at -0.3425 1.516) (layer "F.SilkS")
+    (fp_text reference "D9" (at 0.0625 1.516) (layer "F.SilkS")
       (effects (font (size 1 1) (thickness 0.15)))
     )
@@
     (property "Sheetname" "")
     (attr smd)
-    (fp_text reference "Q3" (at 0 2.4) (layer "F.SilkS")
+    (fp_text reference "Q3" (at 0.25 -2.3) (layer "F.SilkS")
       (effects (font (size 1 1) (thickness 0.15)))
     )
@@
     (property "Sheetname" "")
     (attr smd)
-    (fp_text reference "L2" (at -0.202 1.896 180) (layer "F.SilkS")
-      (effects (font (size 1 1) (thickness 0.15)))
+    (fp_text reference "L2" (at -2.5 1.5 180) (layer "F.SilkS")
+      (effects (font (size 0.8 0.8) (thickness 0.15)))
     )
     (fp_text value "L" (at 0 2.05) (layer "F.Fab")
@@
     (property "Sheetname" "")
     (attr smd)
-    (fp_text reference "Q1" (at 0 2.4) (layer "F.SilkS")
+    (fp_text reference "Q1" (at 0 -2.3) (layer "F.SilkS")
       (effects (font (size 1 1) (thickness 0.15)))
     )
@@
     (property "Sheetname" "")
     (attr smd)
-    (fp_text reference "D11" (at 0.6085 1.614) (layer "F.SilkS")
+    (fp_text reference "D11" (at 1.0625 1.614) (layer "F.SilkS")
       (effects (font (size 1 1) (thickness 0.15)))
     )
@@
     (property "Sheetname" "")
     (attr smd)
-    (fp_text reference "SW1" (at -4.05 0) (layer "F.SilkS")
+    (fp_text reference "SW1" (at -4.05 -2.486) (layer "F.SilkS")
       (effects (font (size 1 1) (thickness 0.15)))
     )
@@
     (property "Sheetname" "")
     (attr smd)
-    (fp_text reference "Q2" (at 0 2.4 90) (layer "F.SilkS")
+    (fp_text reference "Q2" (at 0.75 2.4 90) (layer "F.SilkS")
       (effects (font (size 1 1) (thickness 0.15)))
     )
@@
   (gr_line (start 133.993 56.48476) (end 134.94042 56.38824) (layer "Edge.Cuts") (width 0.1))
   (gr_line (start 125.9031 51.04408) (end 122.436 55.611) (layer "Edge.Cuts") (width 0.1))
+  (gr_text "PCB by Dávid\n\nWarranty void if\nyou can read this.\n\n\n\nVesztettem" (at 130.186 83) (layer "B.SilkS")
+    (effects (font (size 1 1) (thickness 0.15)) (justify mirror))
+  )
+  (gr_text "Rev.A" (at 120 89) (layer "F.SilkS")
+    (effects (font (size 1 1) (thickness 0.15)))
+  )
   (segment (start 123.425 84.175) (end 123.425 83.25) (width 0.4064) (layer "F.Cu") (net 1))
   (segment (start 127.05 95.35) (end 129.947 95.35) (width 0.4064) (layer "F.Cu") (net 1))
