File: hullocsillag.kicad_sch (KiCad schematic)
At the start: 24 parts, among them J1 Conn_01x04, SW1 SW_DPST_x2, U1 STC8G1K08-SOP16

Commit message: hullocsillag
Parts:
- added C3: 10uF, Capacitor_SMD:C_0805_2012Metric, symbol Device:C
- BT1: footprint valami:CR2032_Holder -> karifa:CR2032_Holder
- SW1: footprint valami:SW_Push_K2-1102SP -> karifa:SW_Push_K2-1102SP
Connections:
- net GND: now also C3.2
- net VCC: now also C3.1
Changed lines of the file:
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@@
+    (pin "2")
+  )
+  (symbol (lib_id "Device:C") (at 99.06 49.53 0) (unit 1)
+    (in_bom yes) (on_board yes) (fields_autoplaced)
+    (property "Reference" "C3" (id 0) (at 102.87 48.2599 0)
+      (effects (font (size 1.27 1.27)) (justify left))
+    )
+    (property "Value" "10uF" (id 1) (at 102.87 50.7999 0)
+      (effects (font (size 1.27 1.27)) (justify left))
+    )
+    (property "Footprint" "Capacitor_SMD:C_0805_2012Metric" (id 2) (at 100.0252 53.34 0)
+      (effects (font (size 1.27 1.27)) hide)
+    )
+    (property "Datasheet" "~" (id 3) (at 99.06 49.53 0)
+      (effects (font (size 1.27 1.27)) hide)
+    )
+    (pin "1")
     (pin "2")
   )
@@
     (pin "1")
     (pin "2")
+  )
+  (symbol (lib_id "power:GND") (at 99.06 53.34 0) (unit 1)
+    (in_bom yes) (on_board yes) (fields_autoplaced)
+    (property "Reference" "#PWR0120" (id 0) (at 99.06 59.69 0)
+      (effects (font (size 1.27 1.27)) hide)
+    )
+    (property "Value" "GND" (id 1) (at 99.06 58.42 0))
+    (property "Footprint" "" (id 2) (at 99.06 53.34 0)
+      (effects (font (size 1.27 1.27)) hide)
+    )
+    (property "Datasheet" "" (id 3) (at 99.06 53.34 0)
+      (effects (font (size 1.27 1.27)) hide)
+    )
+    (pin "1")
   )
   (symbol (lib_id "Device:LED") (at 187.96 29.21 270) (unit 1)
@@
       (effects (font (size 1.27 1.27)) (justify left))
     )
-    (property "Footprint" "valami:CR2032_Holder" (id 2) (at 130.175 30.861 90)
+    (property "Footprint" "karifa:CR2032_Holder" (id 2) (at 130.175 30.861 90)
       (effects (font (size 1.27 1.27)) hide)
     )
@@
     (property "Reference" "SW1" (id 0) (at 218.44 81.28 0))
     (property "Value" "SW_DPST_x2" (id 1) (at 218.44 83.82 0))
-    (property "Footprint" "valami:SW_Push_K2-1102SP" (id 2) (at 218.44 87.63 0)
+    (property "Footprint" "karifa:SW_Push_K2-1102SP" (id 2) (at 218.44 87.63 0)
       (effects (font (size 1.27 1.27)) hide)
     )
@@
     (pin "1")
     (pin "2")
+  )
+  (symbol (lib_id "power:VCC") (at 99.06 45.72 0) (unit 1)
+    (in_bom yes) (on_board yes) (fields_autoplaced)
+    (property "Reference" "#PWR0118" (id 0) (at 99.06 49.53 0)
+      (effects (font (size 1.27 1.27)) hide)
+    )
+    (property "Value" "VCC" (id 1) (at 99.06 40.64 0))
+    (property "Footprint" "" (id 2) (at 99.06 45.72 0)
+      (effects (font (size 1.27 1.27)) hide)
+    )
+    (property "Datasheet" "" (id 3) (at 99.06 45.72 0)
+      (effects (font (size 1.27 1.27)) hide)
+    )
+    (pin "1")
   )
   (sheet_instances
@@
       (reference "#PWR0117") (unit 1) (value "VCC") (footprint "")
     )
+    (path "/fccf80e5-f856-491c-ac16-33c399a8d7fe"
+      (reference "#PWR0118") (unit 1) (value "VCC") (footprint "")
+    )
     (path "/97beb115-9240-4226-b6c5-437c3f064a64"
       (reference "#PWR0119") (unit 1) (value "GND") (footprint "")
     )
+    (path "/32eec12e-2416-4397-a503-0957861e91c6"
+      (reference "#PWR0120") (unit 1) (value "GND") (footprint "")
+    )
     (path "/47f7b25e-acd7-4136-8edf-513cdfcedb3a"
-      (reference "BT1") (unit 1) (value "Battery") (footprint "valami:CR2032_Holder")
+      (reference "BT1") (unit 1) (value "Battery") (footprint "karifa:CR2032_Holder")
     )
     (path "/b5491d66-66e5-4963-a31f-7b8012b56406"
@@
       (reference "C2") (unit 1) (value "10uF") (footprint "Capacitor_SMD:C_0805_2012Metric")
     )
+    (path "/0e37a0c7-cb97-4f49-9547-9840b441c59a"
+      (reference "C3") (unit 1) (value "10uF") (footprint "Capacitor_SMD:C_0805_2012Metric")
+    )
     (path "/31b04caa-c4c2-4173-b7a3-7bede720a3d8"
       (reference "D2") (unit 1) (value "LED") (footprint "LED_SMD:LED_0805_2012Metric")
@@
     )
     (path "/de406ba6-034c-4168-9311-f339f51d1cad"
-      (reference "SW1") (unit 1) (value "SW_DPST_x2") (footprint "valami:SW_Push_K2-1102SP")
+      (reference "SW1") (unit 1) (value "SW_DPST_x2") (footprint "karifa:SW_Push_K2-1102SP")
     )
     (path "/700bc6a9-3e36-494a-9775-ec73585b69b4"
