File: karifa.kicad_sch (KiCad schematic)
At the start: 27 parts, among them J1 Conn_01x04, SW1 SW_DPST_x2, U1 STC8G1K08-SOP16

Commit message: proto nyak
Connections:
- net GND: now also U1.8 (GND)
- net P3.1: now also J1.3 (Pin_3)
- net VCC: now also U1.6 (VCC)
Changed lines of the file:
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@@
-    (stroke (width 0) (type default) (color 0 0 0 0))
-  )
-  (wire (pts (xy 96.393 55.626) (xy 96.393 55.753))
     (stroke (width 0) (type default) (color 0 0 0 0))
   )
@@
     (stroke (width 0) (type default) (color 0 0 0 0))
   )
-  (wire (pts (xy 96.266 53.086) (xy 101.473 53.086))
-    (stroke (width 0) (type default) (color 0 0 0 0))
-  )
   (wire (pts (xy 245.11 50.8) (xy 245.11 53.34))
     (stroke (width 0) (type default) (color 0 0 0 0))
@@
     (stroke (width 0) (type default) (color 0 0 0 0))
   )
-  (wire (pts (xy 101.6 55.753) (xy 96.393 55.753))
-    (stroke (width 0) (type default) (color 0 0 0 0))
-  )
   (wire (pts (xy 162.56 21.59) (xy 168.91 21.59))
     (stroke (width 0) (type default) (color 0 0 0 0))
@@
     (stroke (width 0) (type default) (color 0 0 0 0))
   )
+  (wire (pts (xy 96.52 55.88) (xy 101.6 55.88))
+    (stroke (width 0) (type default) (color 0 0 0 0))
+  )
   (wire (pts (xy 128.3208 98.044) (xy 128.3208 100.33))
     (stroke (width 0) (type default) (color 0 0 0 0))
@@
   )
   (wire (pts (xy 168.91 25.4) (xy 168.91 21.59))
+    (stroke (width 0) (type default) (color 0 0 0 0))
+  )
+  (wire (pts (xy 96.52 53.34) (xy 101.6 53.34))
     (stroke (width 0) (type default) (color 0 0 0 0))
   )
@@
     (effects (font (size 1.27 1.27)) (justify left bottom))
   )
-  (label "P3.0" (at 96.3984 53.086 0)
+  (label "P3.0" (at 96.52 53.34 0)
     (effects (font (size 1.27 1.27)) (justify left bottom))
   )
@@
     (effects (font (size 1.27 1.27)) (justify left bottom))
   )
-  (label "P3.1" (at 96.393 55.753 0)
+  (label "P3.1" (at 96.52 55.88 0)
     (effects (font (size 1.27 1.27)) (justify left bottom))
   )
@@
     (pin "2")
   )
-  (symbol (lib_id "power:GND") (at 101.473 58.166 0) (unit 1)
-    (in_bom yes) (on_board yes) (fields_autoplaced)
-    (property "Reference" "#PWR0110" (id 0) (at 101.473 64.516 0)
-      (effects (font (size 1.27 1.27)) hide)
-    )
-    (property "Value" "GND" (id 1) (at 101.473 63.246 0))
-    (property "Footprint" "" (id 2) (at 101.473 58.166 0)
-      (effects (font (size 1.27 1.27)) hide)
-    )
-    (property "Datasheet" "" (id 3) (at 101.473 58.166 0)
+  (symbol (lib_id "power:GND") (at 101.6 58.42 0) (unit 1)
+    (in_bom yes) (on_board yes) (fields_autoplaced)
+    (property "Reference" "#PWR0110" (id 0) (at 101.6 64.77 0)
+      (effects (font (size 1.27 1.27)) hide)
+    )
+    (property "Value" "GND" (id 1) (at 101.6 63.5 0))
+    (property "Footprint" "" (id 2) (at 101.6 58.42 0)
+      (effects (font (size 1.27 1.27)) hide)
+    )
+    (property "Datasheet" "" (id 3) (at 101.6 58.42 0)
       (effects (font (size 1.27 1.27)) hide)
     )
@@
     (pin "2")
   )
+  (symbol (lib_id "power:GND") (at 170.18 113.03 0) (unit 1)
+    (in_bom yes) (on_board yes) (fields_autoplaced)
+    (property "Reference" "#PWR0112" (id 0) (at 170.18 119.38 0)
+      (effects (font (size 1.27 1.27)) hide)
+    )
+    (property "Value" "GND" (id 1) (at 170.18 118.11 0))
+    (property "Footprint" "" (id 2) (at 170.18 113.03 0)
+      (effects (font (size 1.27 1.27)) hide)
+    )
+    (property "Datasheet" "" (id 3) (at 170.18 113.03 0)
+      (effects (font (size 1.27 1.27)) hide)
+    )
+    (pin "1")
+  )
   (symbol (lib_id "Device:LED") (at 187.96 46.99 90) (unit 1)
     (in_bom yes) (on_board yes) (fields_autoplaced)
@@
     (pin "1")
   )
-  (symbol (lib_id "Connector_Generic:Conn_01x04") (at 106.553 53.086 0) (unit 1)
-    (in_bom yes) (on_board yes) (fields_autoplaced)
-    (property "Reference" "J1" (id 0) (at 109.22 53.0859 0)
-      (effects (font (size 1.27 1.27)) (justify left))
-    )
-    (property "Value" "Conn_01x04" (id 1) (at 109.22 55.6259 0)
-      (effects (font (size 1.27 1.27)) (justify left))
-    )
-    (property "Footprint" "Connector_PinHeader_2.54mm:PinHeader_1x04_P2.54mm_Vertical" (id 2) (at 106.553 53.086 0)
-      (effects (font (size 1.27 1.27)) hide)
-    )
-    (property "Datasheet" "~" (id 3) (at 106.553 53.086 0)
+  (symbol (lib_id "Connector_Generic:Conn_01x04") (at 106.68 53.34 0) (unit 1)
+    (in_bom yes) (on_board yes) (fields_autoplaced)
+    (property "Reference" "J1" (id 0) (at 109.347 53.3399 0)
+      (effects (font (size 1.27 1.27)) (justify left))
+    )
+    (property "Value" "Conn_01x04" (id 1) (at 109.347 55.8799 0)
+      (effects (font (size 1.27 1.27)) (justify left))
+    )
+    (property "Footprint" "Connector_PinHeader_2.54mm:PinHeader_1x04_P2.54mm_Vertical" (id 2) (at 106.68 53.34 0)
+      (effects (font (size 1.27 1.27)) hide)
+    )
+    (property "Datasheet" "~" (id 3) (at 106.68 53.34 0)
       (effects (font (size 1.27 1.27)) hide)
     )
@@
     (pin "1")
     (pin "2")
+  )
+  (symbol (lib_id "power:VCC") (at 170.18 72.39 0) (unit 1)
+    (in_bom yes) (on_board yes) (fields_autoplaced)
+    (property "Reference" "#PWR0111" (id 0) (at 170.18 76.2 0)
+      (effects (font (size 1.27 1.27)) hide)
+    )
+    (property "Value" "VCC" (id 1) (at 170.18 67.31 0))
+    (property "Footprint" "" (id 2) (at 170.18 72.39 0)
+      (effects (font (size 1.27 1.27)) hide)
+    )
+    (property "Datasheet" "" (id 3) (at 170.18 72.39 0)
+      (effects (font (size 1.27 1.27)) hide)
+    )
+    (pin "1")
   )
   (symbol (lib_id "Device:LED") (at 207.01 46.99 90) (unit 1)
@@
     (pin "1")
   )
-  (symbol (lib_id "power:VCC") (at 101.473 50.546 0) (unit 1)
-    (in_bom yes) (on_board yes) (fields_autoplaced)
-    (property "Reference" "#PWR0102" (id 0) (at 101.473 54.356 0)
-      (effects (font (size 1.27 1.27)) hide)
-    )
-    (property "Value" "VCC" (id 1) (at 101.473 45.72 0))
-    (property "Footprint" "" (id 2) (at 101.473 50.546 0)
-      (effects (font (size 1.27 1.27)) hide)
-    )
-    (property "Datasheet" "" (id 3) (at 101.473 50.546 0)
+  (symbol (lib_id "power:VCC") (at 101.6 50.8 0) (unit 1)
+    (in_bom yes) (on_board yes) (fields_autoplaced)
+    (property "Reference" "#PWR0102" (id 0) (at 101.6 54.61 0)
+      (effects (font (size 1.27 1.27)) hide)
+    )
+    (property "Value" "VCC" (id 1) (at 101.6 45.974 0))
+    (property "Footprint" "" (id 2) (at 101.6 50.8 0)
+      (effects (font (size 1.27 1.27)) hide)
+    )
+    (property "Datasheet" "" (id 3) (at 101.6 50.8 0)
       (effects (font (size 1.27 1.27)) hide)
     )
@@
       (reference "#PWR0110") (unit 1) (value "GND") (footprint "")
     )
+    (path "/ba9d3f38-ddab-4d58-919a-28c0eaa6d3b7"
+      (reference "#PWR0111") (unit 1) (value "VCC") (footprint "")
+    )
+    (path "/736018fa-45a8-4e79-b4fc-6ce85c731ce4"
+      (reference "#PWR0112") (unit 1) (value "GND") (footprint "")
+    )
     (path "/47f7b25e-acd7-4136-8edf-513cdfcedb3a"

Commit message: nyakterv majdnem kesz
Parts:
- removed D1: LED_RGB, LED_SMD:LED_RGB_5050-6, symbol Device:LED_RGB
- added D1: LED_ARGB, LED_SMD:LED_RGB_Wuerth-PLCC4_3.2x2.8mm_150141M173100, symbol Device:LED_ARGB
- added L1, L2, L3: L, Inductor_SMD:L_1008_2520Metric, symbol Device:L
- added Q1, Q2, Q3: AO3401A, Package_TO_SOT_SMD:SOT-23, symbol Transistor_FET:AO3401A
- BT1: footprint Battery:BatteryHolder_ComfortableElectronic_CH273-2450_1x2450 -> karifa:CR2032_Holder
- J1: footprint Connector_PinHeader_2.54mm:PinHeader_1x04_P2.54mm_Vertical -> Connector_PinHeader_1.27mm:PinHeader_1x04_P1.27mm_Vertical
- R1, R2, R3, R4, R5, R6, R7, R8, R9: footprint Resistor_SMD:R_0805_2012Metric -> Resistor_SMD:R_0603_1608Metric
Connections:
- net GND: now also D1.1 (A), L1.2, L2.2, L3.2; no longer R1.2, R2.2, R3.2
- net P1.6: now also R2.2, Q2.1 (G); no longer R9.2
- net VCC: now also R1.1, R2.1, R3.1, Q1.2 (S), Q2.2 (S), Q3.2 (S)
- net P1.7: now reaches U1.4 (P1.7)
- net P1.7: now also R9.2
- net P5.4: now reaches U1.5 (P5.4)
- net P5.4: now also R3.2, Q3.1 (G)
- net P5.5: now reaches U1.7 (P5.5)
- net P5.5: now also R1.2, Q1.1 (G)
- new net: D1.2 (RK), L2.1, Q2.3 (D)
- new net: D1.3 (GK), L3.1, Q3.3 (D)
- new net: D1.4 (BK), L1.1, Q1.3 (D)
Other:
- moved on the sheet: J1

Commit message: nyakterv haladas
Parts:
- added C2, C3: 10uF, Capacitor_SMD:C_0805_2012Metric, symbol Device:C
- C1: value C -> 100nF
- R1, R2, R3: value R -> 100k
- R4, R5, R6, R7, R8, R9: value R -> 1k
Connections:
- net GND: now also C2.2, C3.2
- net VCC: now also C2.1, C3.1

Commit message: panelizacio
Parts:
- added T1: Tab, kikit:Tab, symbol kikit:Tab
Changed lines of the file:
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@@
     (pin "2")
+  )
+  (symbol (lib_id "kikit:Tab") (at 100.33 114.3 0) (unit 1)
+    (in_bom no) (on_board yes) (fields_autoplaced)
+    (property "Reference" "T1" (id 0) (at 105.41 112.3949 0)
+      (effects (font (size 1.27 1.27)) (justify left))
+    )
+    (property "Value" "Tab" (id 1) (at 105.41 114.9349 0)
+      (effects (font (size 1.27 1.27)) (justify left))
+    )
+    (property "Footprint" "kikit:Tab" (id 2) (at 100.33 114.3 0)
+      (effects (font (size 1.27 1.27)) hide)
+    )
+    (property "Datasheet" "" (id 3) (at 100.33 114.3 0)
+      (effects (font (size 1.27 1.27)) hide)
+    )
   )
   (symbol (lib_id "Device:L") (at 53.34 52.07 0) (unit 1)
@@
       (reference "SW1") (unit 1) (value "SW_DPST_x2") (footprint "karifa:SW_Push_K2-1102SP")
     )
+    (path "/0b72e181-2db7-4b27-9232-922c0199bb96"
+      (reference "T1") (unit 1) (value "Tab") (footprint "kikit:Tab")
+    )
     (path "/700bc6a9-3e36-494a-9775-ec73585b69b4"

Commit message: javitasok
Parts:
- Q1, Q2, Q3: footprint Package_TO_SOT_SMD:SOT-23 -> sajat:SOT-23
- SW1: footprint karifa:SW_Push_K2-1102SP -> sajat:SW_Push_K2-1102SP
Changed lines of the file:
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@@
     (property "Reference" "Q3" (id 0) (at 44.45 62.23 90))
     (property "Value" "AO3401A" (id 1) (at 44.45 64.77 90))
-    (property "Footprint" "Package_TO_SOT_SMD:SOT-23" (id 2) (at 42.545 67.31 0)
+    (property "Footprint" "sajat:SOT-23" (id 2) (at 42.545 67.31 0)
       (effects (font (size 1.27 1.27) italic) (justify left) hide)
     )
@@
     (property "Reference" "Q2" (id 0) (at 44.45 38.1 90))
     (property "Value" "AO3401A" (id 1) (at 44.45 40.64 90))
-    (property "Footprint" "Package_TO_SOT_SMD:SOT-23" (id 2) (at 42.545 43.18 0)
+    (property "Footprint" "sajat:SOT-23" (id 2) (at 42.545 43.18 0)
       (effects (font (size 1.27 1.27) italic) (justify left) hide)
     )
@@
     (property "Reference" "SW1" (id 0) (at 218.44 81.28 0))
     (property "Value" "SW_DPST_x2" (id 1) (at 218.44 83.82 0))
-    (property "Footprint" "karifa:SW_Push_K2-1102SP" (id 2) (at 218.44 87.63 0)
+    (property "Footprint" "sajat:SW_Push_K2-1102SP" (id 2) (at 218.44 87.63 0)
       (effects (font (size 1.27 1.27)) hide)
     )
@@
     (property "Reference" "Q1" (id 0) (at 41.91 87.63 90))
     (property "Value" "AO3401A" (id 1) (at 41.91 90.17 90))
-    (property "Footprint" "Package_TO_SOT_SMD:SOT-23" (id 2) (at 40.005 92.71 0)
+    (property "Footprint" "sajat:SOT-23" (id 2) (at 40.005 92.71 0)
       (effects (font (size 1.27 1.27) italic) (justify left) hide)
     )
@@
     )
     (path "/fc90615f-14ab-4e28-a4dd-78e4c9052225"
-      (reference "Q1") (unit 1) (value "AO3401A") (footprint "Package_TO_SOT_SMD:SOT-23")
+      (reference "Q1") (unit 1) (value "AO3401A") (footprint "sajat:SOT-23")
     )
     (path "/8ad2b27f-56c4-4507-95fe-ff61e05d0e5d"
-      (reference "Q2") (unit 1) (value "AO3401A") (footprint "Package_TO_SOT_SMD:SOT-23")
+      (reference "Q2") (unit 1) (value "AO3401A") (footprint "sajat:SOT-23")
     )
     (path "/17a5f37d-34c8-4ccd-b3cd-7b199e521964"
-      (reference "Q3") (unit 1) (value "AO3401A") (footprint "Package_TO_SOT_SMD:SOT-23")
+      (reference "Q3") (unit 1) (value "AO3401A") (footprint "sajat:SOT-23")
     )
     (path "/23172657-7dcf-40a6-be57-7a2d6a0ef71d"
@@
     )
     (path "/de406ba6-034c-4168-9311-f339f51d1cad"
-      (reference "SW1") (unit 1) (value "SW_DPST_x2") (footprint "karifa:SW_Push_K2-1102SP")
+      (reference "SW1") (unit 1) (value "SW_DPST_x2") (footprint "sajat:SW_Push_K2-1102SP")
     )
     (path "/0b72e181-2db7-4b27-9232-922c0199bb96"
