File: karifa.kicad_sch (KiCad schematic)
At the start: 24 parts, among them J1 Conn_01x04, SW1 SW_DPST_x2, U1 STC8G1K08-SOP16

Commit message: hullocsillag
Parts:
- added T1, T? (x2): Tab, kikit:Tab, symbol kikit:Tab
- SW1: footprint valami:SW_Push_K2-1102SP -> karifa:SW_Push_K2-1102SP
Changed lines of the file:
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@@
     (pin "2")
+  )
+  (symbol (lib_id "kikit:Tab") (at 250.19 125.73 0) (unit 1)
+    (in_bom no) (on_board yes) (fields_autoplaced)
+    (property "Reference" "T?" (id 0) (at 255.27 123.8249 0)
+      (effects (font (size 1.27 1.27)) (justify left))
+    )
+    (property "Value" "Tab" (id 1) (at 255.27 126.3649 0)
+      (effects (font (size 1.27 1.27)) (justify left))
+    )
+    (property "Footprint" "kikit:Tab" (id 2) (at 250.19 125.73 0)
+      (effects (font (size 1.27 1.27)) hide)
+    )
+    (property "Datasheet" "" (id 3) (at 250.19 125.73 0)
+      (effects (font (size 1.27 1.27)) hide)
+    )
   )
   (symbol (lib_id "power:GND") (at 118.11 53.34 0) (unit 1)
@@
     (pin "1")
   )
+  (symbol (lib_id "kikit:Tab") (at 252.73 118.11 0) (unit 1)
+    (in_bom no) (on_board yes) (fields_autoplaced)
+    (property "Reference" "T1" (id 0) (at 257.81 116.2049 0)
+      (effects (font (size 1.27 1.27)) (justify left))
+    )
+    (property "Value" "Tab" (id 1) (at 257.81 118.7449 0)
+      (effects (font (size 1.27 1.27)) (justify left))
+    )
+    (property "Footprint" "kikit:Tab" (id 2) (at 252.73 118.11 0)
+      (effects (font (size 1.27 1.27)) hide)
+    )
+    (property "Datasheet" "" (id 3) (at 252.73 118.11 0)
+      (effects (font (size 1.27 1.27)) hide)
+    )
+  )
+  (symbol (lib_id "kikit:Tab") (at 234.95 125.73 0) (unit 1)
+    (in_bom no) (on_board yes) (fields_autoplaced)
+    (property "Reference" "T?" (id 0) (at 240.03 123.8249 0)
+      (effects (font (size 1.27 1.27)) (justify left))
+    )
+    (property "Value" "Tab" (id 1) (at 240.03 126.3649 0)
+      (effects (font (size 1.27 1.27)) (justify left))
+    )
+    (property "Footprint" "kikit:Tab" (id 2) (at 234.95 125.73 0)
+      (effects (font (size 1.27 1.27)) hide)
+    )
+    (property "Datasheet" "" (id 3) (at 234.95 125.73 0)
+      (effects (font (size 1.27 1.27)) hide)
+    )
+  )
   (symbol (lib_id "Device:LED") (at 207.01 46.99 90) (unit 1)
     (in_bom yes) (on_board yes) (fields_autoplaced)
@@
     (property "Reference" "SW1" (id 0) (at 218.44 81.28 0))
     (property "Value" "SW_DPST_x2" (id 1) (at 218.44 83.82 0))
-    (property "Footprint" "valami:SW_Push_K2-1102SP" (id 2) (at 218.44 87.63 0)
+    (property "Footprint" "karifa:SW_Push_K2-1102SP" (id 2) (at 218.44 87.63 0)
       (effects (font (size 1.27 1.27)) hide)
     )
@@
     )
     (path "/de406ba6-034c-4168-9311-f339f51d1cad"
-      (reference "SW1") (unit 1) (value "SW_DPST_x2") (footprint "valami:SW_Push_K2-1102SP")
+      (reference "SW1") (unit 1) (value "SW_DPST_x2") (footprint "karifa:SW_Push_K2-1102SP")
+    )
+    (path "/bfebb9ae-e5e7-4836-9610-4e5d135a335f"
+      (reference "T1") (unit 1) (value "Tab") (footprint "kikit:Tab")
+    )
+    (path "/1095e108-a30a-428e-990a-ac9325d5c3fd"
+      (reference "T?") (unit 1) (value "Tab") (footprint "kikit:Tab")
+    )
+    (path "/c58a6ff2-94c6-4905-a938-4a10820232f2"
+      (reference "T?") (unit 1) (value "Tab") (footprint "kikit:Tab")
     )
     (path "/700bc6a9-3e36-494a-9775-ec73585b69b4"
